File: schematic_diagram_3.sch (KiCad schematic (older format))
At the start: 12 parts, among them J1 XLR3_Switched, J2 XLR3_Switched, J3 Conn_01x02_Female, U1 74LS04, U2 74AUC2G08, U3 74LVC2G02

Commit message: Add files via upload
Parts:
- U1, U2, U3: footprint (none) -> Package_DIP:DIP-14_W7.62mm
Changed lines of the file:
@@
 F 0 "U3" H 6375 3667 50  0000 C CNN
 F 1 "74LVC2G02" H 6375 3576 50  0000 C CNN
-F 2 "" H 6400 3400 50  0001 C CNN
+F 2 "Package_DIP:DIP-14_W7.62mm" H 6400 3400 50  0001 C CNN
 F 3 "http://www.ti.com/lit/sg/scyt129e/scyt129e.pdf" H 6400 3400 50  0001 C CNN
 	1    6400 3400
@@
 F 0 "U3" H 6375 4317 50  0000 C CNN
 F 1 "74LVC2G02" H 6375 4226 50  0000 C CNN
-F 2 "" H 6400 4050 50  0001 C CNN
+F 2 "Package_DIP:DIP-14_W7.62mm" H 6400 4050 50  0001 C CNN
 F 3 "http://www.ti.com/lit/sg/scyt129e/scyt129e.pdf" H 6400 4050 50  0001 C CNN
 	2    6400 4050
@@
 F 0 "U1" H 4650 3617 50  0000 C CNN
 F 1 "74LS04" H 4650 3526 50  0000 C CNN
-F 2 "" H 4650 3300 50  0001 C CNN
+F 2 "Package_DIP:DIP-14_W7.62mm" H 4650 3300 50  0001 C CNN
 F 3 "http://www.ti.com/lit/gpn/sn74LS04" H 4650 3300 50  0001 C CNN
 	1    4650 3300
@@
 F 0 "U2" H 5625 3617 50  0000 C CNN
 F 1 "74AUC2G08" H 5625 3526 50  0000 C CNN
-F 2 "" H 5650 3350 50  0001 C CNN
+F 2 "Package_DIP:DIP-14_W7.62mm" H 5650 3350 50  0001 C CNN
 F 3 "http://www.ti.com/lit/sg/scyt129e/scyt129e.pdf" H 5650 3350 50  0001 C CNN
 	2    5650 3350
@@
 F 0 "U2" H 5575 4367 50  0000 C CNN
 F 1 "74AUC2G08" H 5575 4276 50  0000 C CNN
-F 2 "" H 5600 4100 50  0001 C CNN
+F 2 "Package_DIP:DIP-14_W7.62mm" H 5600 4100 50  0001 C CNN
 F 3 "http://www.ti.com/lit/sg/scyt129e/scyt129e.pdf" H 5600 4100 50  0001 C CNN
 	1    5600 4100
